File: PCB/60_FN.brd (EAGLE design)
At the start: 285.2 x 115.3 mm, 75 parts

Commit message: Add files via upload
Parts:
- removed U1: (no value), MCU:LQFP100
- added U2: (no value), MCU:LQFP100
Other:
- board size 285.2 x 115.3 mm -> 285.2 x 117.6 mm
